File: electronique/moon-rover.sch (EAGLE design)
At the start: 85 parts

Commit message: LL: définition des ordres décrits par la documentation, implémentation des ordres de locomotion
Parts:
- added C22, C23: (no value), 1NTech_RLCD:CPOL-EUE2.5-6
- added DC4: R-78C9.0-1.0, dc-dc-converter:R-78C9.0-1.0
Connections:
- new net +9V_AV: AX12_DIRECTION.2, C20.+, C22.+, DC4.VOUT
- net +12V: now also C23.+, DC4.VIN
- net +9V: no longer AX12_DIRECTION.2, C20.+
- net GND: now also C22.-, C23.-, DC4.GND
Other:
- moved on the sheet: PHARES_AR_D, PHARES_AR_G, PHARES_AV_D, PHARES_AV_G, RASPBERRY_PI

Commit message: LL: debug + config + maj de l'élec
Parts:
- removed C14: 10n, 1NTech_RLCD:C-EU050-024X044
- removed C15, C16: 1µF, 1NTech_RLCD:CPOL-EUE2.5-5
- removed C17, C18: 220µF, 1NTech_RLCD:CPOL-EUE3.5-8
- removed R3, R4: 10k, 1NTech_RLCD:R-EU_0204/7
- added C24, C25: 100n, 1NTech_RLCD:C-EU050-024X044
- added R28, R29: 10k, 1NTech_RLCD:R-EU_0204/7
- C11, C12: value 10n -> 100n
- C13: value 10n -> (none); device 1NTech_RLCD:C-EU050-024X044 -> resistor:CPOL-EUE5-13
- PONT_H_M_D, PONT_H_M_G: value LM18200T -> L298; device national-semiconductor:LM18200T -> st-microelectronics:L298; MPN (none) -> L298N; OC_FARNELL (none) -> 1589425; OC_NEWARK (none) -> 32M1527
- R14, R16, R18, R22, R24: value ? -> 270
- R15, R17, R19, R20, R21, R27: value ? -> 330
- R23: value ? -> 100
- R25: value ? -> 15
- R26: value ? -> 820
Connections:
- removed net MOTEUR_D_DIR: PONT_H_M_D.DIRECTION, R4.2, U$2.4/CAN0-RX/SDA2/PWM
- removed net MOTEUR_D_PWM: PONT_H_M_D.PWM, R3.2, U$2.6/PWM
- removed net MOTEUR_G_DIR: PONT_H_M_G.DIRECTION, R2.2, U$2.3/CAN0-TX/SCL2/PWM
- removed net MOTEUR_G_PWM: PONT_H_M_G.PWM, R1.2, U$2.5/PWM
- removed net N$1: C11.2, PONT_H_M_G.BOOTSTRAP1
- removed net N$3: C12.1, PONT_H_M_G.BOOTSTRAP2
- removed net N$6: C13.2, PONT_H_M_D.BOOTSTRAP1
- removed net N$7: C14.1, PONT_H_M_D.BOOTSTRAP2
- new net MOTEUR_D_A: PONT_H_M_D.INPUT1, PONT_H_M_D.INPUT4, R2.2, U$2.4/CAN0-RX/SDA2/PWM
- new net MOTEUR_D_B: PONT_H_M_D.INPUT2, PONT_H_M_D.INPUT3, R1.2, U$2.6/PWM
- new net MOTEUR_G_A: PONT_H_M_G.INPUT1, PONT_H_M_G.INPUT4, R29.2, U$2.3/CAN0-TX/SCL2/PWM
- new net MOTEUR_G_B: PONT_H_M_G.INPUT2, PONT_H_M_G.INPUT3, R28.2, U$2.5/PWM
- net +12V: now also C12.1, C13.+, C25.1; no longer C15.+, C16.+, C17.+, C18.+
- net +5V: now also C11.2, C24.2, PONT_H_M_D.ENABLE_A, PONT_H_M_D.ENABLE_B, PONT_H_M_D.VCC, PONT_H_M_G.ENABLE_A, PONT_H_M_G.ENABLE_B, PONT_H_M_G.VCC
- net GND: now also C11.1, C12.2, C13.-, C24.1, C25.2, PONT_H_M_D.SEN_A, PONT_H_M_D.SEN_B, PONT_H_M_G.SEN_A, PONT_H_M_G.SEN_B, R28.1, R29.1; no longer C15.-, C16.-, C17.-, C18.-, PONT_H_M_D.BREAK, PONT_H_M_G.BREAK, R3.1, R4.1
- net MOTEUR_D_+: now also PONT_H_M_D.OUT1, PONT_H_M_D.OUT4; no longer C13.1, PONT_H_M_D.OUTPUT1
- net MOTEUR_D_-: now also PONT_H_M_D.OUT2, PONT_H_M_D.OUT3; no longer C14.2, PONT_H_M_D.OUTPUT2
- net MOTEUR_G_+: now also PONT_H_M_G.OUT1, PONT_H_M_G.OUT4; no longer C11.1, PONT_H_M_G.OUTPUT1
- net MOTEUR_G_-: now also PONT_H_M_G.OUT2, PONT_H_M_G.OUT3; no longer C12.2, PONT_H_M_G.OUTPUT2
Other:
- moved on the sheet: C11, C12, R1, R2
